Commit message: Move manual pelvis collisions to dedicated file

File: config/srdf/disable_collisions/kangaroo_no-arms_with-pelvis.srdf.xacro (robot description, xacro)
@@ -2,4 +2,5 @@
 <robot name="kangaroo" xmlns:xacro="http://ros.org/wiki/xacro">
   <xacro:include filename="$(find kangaroo_moveit_config)/config/srdf/disable_collisions/kangaroo_no-arms_no-pelvis.srdf.xacro" />
+  <xacro:include filename="$(find kangaroo_moveit_config)/config/srdf/disable_collisions/manual_pelvis_collisions.srdf.xacro" />
     <disable_collisions link1="arm_cover_left_cover_link" link2="back_handle" reason="Never"/>
     <disable_collisions link1="arm_cover_left_cover_link" link2="pelvis_1_link" reason="Never"/>

File: config/srdf/kangaroo.srdf.xacro (robot description, xacro)
@@ -170,18 +170,4 @@
     <!-- NOTE: from here onwards there are manual disabled collision -->
     <!-- TODO: This needs to be handled properly with the update.sh script -->
-    <xacro:macro name="back_handle_leg_disable_collisions" params="side">
-        <disable_collisions link1="back_handle" link2="leg_${side}_1_link" reason="Never"/>
-    </xacro:macro>
-    <xacro:back_handle_leg_disable_collisions side="left"/>
-    <xacro:back_handle_leg_disable_collisions side="right"/>
-    <xacro:if value="${has_pelvis}">
-        <xacro:macro name="pelvis_leg_disable_collisions" params="side">
-            <disable_collisions link1="pelvis_base_link" link2="leg_${side}_1_link" reason="Never"/>
-            <disable_collisions link1="pelvis_1_link" link2="leg_${side}_1_link" reason="Never"/>
-            <disable_collisions link1="pelvis_2_link" link2="leg_${side}_1_link" reason="Never"/>
-        </xacro:macro>
-        <xacro:pelvis_leg_disable_collisions side="left"/>
-        <xacro:pelvis_leg_disable_collisions side="right"/>
-    </xacro:if>
     <xacro:macro name="leg_closed_loop_disable_collisions" params="side">
         <disable_collisions link1="base_link"               link2="leg_${side}_femur_link" reason="Never"/>
