Commit message: Move manual leg collisions to dedicated file

File: config/srdf/disable_collisions/kangaroo_no-arms_no-pelvis_detachable.srdf.xacro (robot description, xacro)
@@ -1,4 +1,5 @@
 <?xml version="1.0" ?>
 <robot name="kangaroo" xmlns:xacro="http://ros.org/wiki/xacro">
+    <xacro:include filename="$(find kangaroo_moveit_config)/config/srdf/disable_collisions/manual_legs_collision.srdf.xacro"/>
     <disable_collisions link1="ankle_left_ft_sensor_link" link2="arm_cover_left_cover_link" reason="Never"/>
     <disable_collisions link1="ankle_left_ft_sensor_link" link2="arm_cover_right_cover_link" reason="Never"/>

File: config/srdf/disable_collisions/kangaroo_no-arms_no-pelvis_fixed.srdf.xacro (robot description, xacro)
@@ -1,4 +1,5 @@
 <?xml version="1.0" ?>
 <robot name="kangaroo" xmlns:xacro="http://ros.org/wiki/xacro">
+    <xacro:include filename="$(find kangaroo_moveit_config)/config/srdf/disable_collisions/manual_legs_collision.srdf.xacro" />
     <disable_collisions link1="arm_cover_left_cover_link" link2="arm_cover_right_cover_link" reason="Never"/>
     <disable_collisions link1="arm_cover_left_cover_link" link2="base_link" reason="Never"/>

File: config/srdf/disable_collisions/kangaroo_no-arms_with-pelvis.srdf.xacro (robot description, xacro)
@@ -2,5 +2,4 @@
 <robot name="kangaroo" xmlns:xacro="http://ros.org/wiki/xacro">
   <xacro:include filename="$(find kangaroo_moveit_config)/config/srdf/disable_collisions/kangaroo_no-arms_no-pelvis.srdf.xacro" />
-  <xacro:include filename="$(find kangaroo_moveit_config)/config/srdf/disable_collisions/manual_pelvis_collisions.srdf.xacro" />
     <disable_collisions link1="arm_cover_left_cover_link" link2="back_handle" reason="Never"/>
     <disable_collisions link1="arm_cover_left_cover_link" link2="pelvis_1_link" reason="Never"/>

File: config/srdf/disable_collisions/kangaroo_no-arms_with-pelvis_detachable.srdf.xacro (robot description, xacro)
@@ -2,4 +2,5 @@
 <robot name="kangaroo" xmlns:xacro="http://ros.org/wiki/xacro">
   <xacro:include filename="$(find kangaroo_moveit_config)/config/srdf/disable_collisions/kangaroo_no-arms_no-pelvis_detachable.srdf.xacro" />
+  <xacro:include filename="$(find kangaroo_moveit_config)/config/srdf/disable_collisions/manual_pelvis_collisions.srdf.xacro" />
     <disable_collisions link1="ankle_left_ft_sensor_link" link2="back_handle" reason="Never"/>
     <disable_collisions link1="ankle_left_ft_sensor_link" link2="pelvis_1_link" reason="Never"/>

File: config/srdf/disable_collisions/kangaroo_no-arms_with-pelvis_fixed.srdf.xacro (robot description, xacro)
@@ -2,4 +2,5 @@
 <robot name="kangaroo" xmlns:xacro="http://ros.org/wiki/xacro">
   <xacro:include filename="$(find kangaroo_moveit_config)/config/srdf/disable_collisions/kangaroo_no-arms_no-pelvis_fixed.srdf.xacro" />
+  <xacro:include filename="$(find kangaroo_moveit_config)/config/srdf/disable_collisions/manual_pelvis_collisions.srdf.xacro" />
     <disable_collisions link1="arm_cover_left_cover_link" link2="back_handle" reason="Never"/>
     <disable_collisions link1="arm_cover_left_cover_link" link2="pelvis_1_link" reason="Never"/>

File: config/srdf/kangaroo.srdf.xacro (robot description, xacro)
@@ -168,20 +168,3 @@
     <xacro:property name="base_arm_token" value="${arm_type if has_arm else 'no-arms'}"/>
     <xacro:include filename="$(find kangaroo_moveit_config)/config/srdf/disable_collisions/${robot}_${base_arm_token}_${'with-pelvis' if has_pelvis else 'no-pelvis'}_${feet_type}.srdf.xacro" />
-    <!-- NOTE: from here onwards there are manual disabled collision -->
-    <!-- TODO: This needs to be handled properly with the update.sh script -->
-    <xacro:macro name="leg_closed_loop_disable_collisions" params="side">
-        <disable_collisions link1="base_link"               link2="leg_${side}_femur_link" reason="Never"/>
-        <disable_collisions link1="leg_${side}_1_link"      link2="leg_${side}_femur_link" reason="Never"/>
-        <disable_collisions link1="leg_${side}_3_link"      link2="leg_${side}_femur_link" reason="Never"/>
-        <disable_collisions link1="leg_${side}_3_link"      link2="leg_${side}_knee_link"  reason="Never"/>
-        <disable_collisions link1="leg_${side}_4_link"      link2="leg_${side}_femur_link" reason="Never"/>
-        <disable_collisions link1="leg_${side}_4_link"      link2="leg_${side}_knee_link"  reason="Never"/>
-        <disable_collisions link1="leg_${side}_5_link"      link2="leg_${side}_femur_link" reason="Never"/>
-        <disable_collisions link1="leg_${side}_5_link"      link2="leg_${side}_knee_link"  reason="Never"/>
-        <disable_collisions link1="leg_${side}_femur_link"  link2="leg_${side}_knee_link"  reason="Never"/>
-    </xacro:macro>
-    <xacro:leg_closed_loop_disable_collisions side="left"/>
-    <xacro:leg_closed_loop_disable_collisions side="right"/>
-    <disable_collisions link1="leg_right_1_link" link2="leg_left_1_link" reason="Never"/>
-    <disable_collisions link1="leg_right_1_link" link2="leg_right_3_link" reason="Never"/>
 </robot>
